File: hardware/EuroPi-X/kicad/neopixels/neopixels.kicad_sch (KiCad schematic)
At the start: 16 parts, among them J1 Conn_01x04_Pin, Q1 BSS138

Commit message: kicad save
Parts:
- D5: JLCPCB Rotation Offset (none) -> 90
Changed lines of the file:
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@@
+      (effects (font (size 1.27 1.27)) hide)
+    )
+    (property "JLCPCB Rotation Offset" "90" (at 88.9 85.09 0)
       (effects (font (size 1.27 1.27)) hide)
     )
