File: hardware/EuroPi-X/development/analogue_input/analogue_input.kicad_sch (KiCad schematic)
At the start: 28 parts, among them J10 Thonkiconn_Mono_Jack, J3 Thonkiconn_Mono_Jack, J4 Thonkiconn_Mono_Jack, J6 Conn_01x06_Pin, J9 Thonkiconn_Mono_Jack, U10 MCP3428, U3 LM4040DBZ-10, U9 MCP6004

Commit message: rearrange fully
Parts:
- removed J6: Conn_01x06_Pin, Connector_PinHeader_2.54mm:PinHeader_1x06_P2.54mm_Vertical, symbol Connector:Conn_01x06_Pin
- removed R26, R39, R40: 15K, Resistor_SMD:R_0402_1005Metric, symbol Device:R
- added J5: Conn_02x05_Odd_Even, allen-synthesis:power-header-10-pin-unlabelled, symbol Connector_Generic:Conn_02x05_Odd_Even
- added J6: Conn_01x02_Pin, Connector_PinHeader_2.54mm:PinHeader_1x02_P2.54mm_Vertical, symbol Connector:Conn_01x02_Pin
- added J7: Conn_01x04_Pin, Connector_PinHeader_2.54mm:PinHeader_1x04_P2.54mm_Vertical, symbol Connector:Conn_01x04_Pin
- added R25 (x4): 1K, Resistor_SMD:R_0402_1005Metric, symbol Device:R
- added R25 (x3): 15K, Resistor_SMD:R_0402_1005Metric, symbol Device:R
Connections:
- net +3.3V: now also J7.2 (Pin_2)
- net -12V: now also J5.1 (Pin_1), J5.2 (Pin_2)
- net ADC_INPUT_1: now also R25.2; no longer R25.2
- net ADC_INPUT_2: now also R25.2
- net ADC_INPUT_3: now also R25.2
- net ADC_INPUT_4: now also R25.2
- net Earth: now also U9.10 (+), U9.12 (+), U9.3 (+), U9.5 (+), J5.3 (Pin_3), J5.4 (Pin_4), J5.5 (Pin_5), J5.6 (Pin_6), J5.7 (Pin_7), J5.8 (Pin_8), J6.1 (Pin_1), J7.1 (Pin_1); no longer U9.13 (-), U9.2 (-), U9.6 (-), U9.9 (-)
- net I2C0_SCL: now also J7.3 (Pin_3)
- net I2C0_SDA: now also J7.4 (Pin_4)
- net INPUT_DETECT: now also J6.2 (Pin_2)
- net at R22.2, R23.2: now also U9.9 (-), R25.1; no longer U9.10 (+)
- net at R35.2, R36.2: now also U9.13 (-), R25.1; no longer U9.12 (+)
- net at R20.2, R21.2, R25.1: now also U9.2 (-); no longer U9.3 (+)
- net at R37.2, R38.2: now also U9.6 (-), R25.1; no longer U9.5 (+)
- new net: R25.1, R25.2 (x4)
- new net +12V: J5.10 (Pin_10), J5.9 (Pin_9)
Other:
- note added: "15K and 1K used to remain within E6 standard series values only"
- note added: "It is then inverted and attenuated by 0.15x resulting in a range of +3.2V to 0V, which is a safe range to feed into the +3.3V tolerant ADC input."
- note removed: "It is then inverted and attenuated by 0.15x resulting in a range of +3V to 0V, which is a safe range to feed into the +3.3V tolerant ADC input."
- moved on the sheet: R25

Commit message: analogue input dev board update
Parts:
- removed J10, J3, J4, J9: Thonkiconn_Mono_Jack, allen-synthesis:jack-thonkiconn-mono, symbol Eurorack:Thonkiconn_Mono_Jack
- removed J5: Conn_02x05_Odd_Even, allen-synthesis:power-header-10-pin-unlabelled, symbol Connector_Generic:Conn_02x05_Odd_Even
- removed J6: Conn_01x02_Pin, Connector_PinHeader_2.54mm:PinHeader_1x02_P2.54mm_Vertical, symbol Connector:Conn_01x02_Pin
- removed J7: Conn_01x04_Pin, Connector_PinHeader_2.54mm:PinHeader_1x04_P2.54mm_Vertical, symbol Connector:Conn_01x04_Pin
- removed R20 (x4): 100K, Resistor_SMD:R_0402_1005Metric, symbol Device:R
- added J1, J2: Conn_01x06_Pin, Connector_PinHeader_2.54mm:PinHeader_1x06_P2.54mm_Vertical, symbol Connector:Conn_01x06_Pin
Connections:
- net -10VREF: now also J2.5 (Pin_5)
- net -12V: now also J1.3 (Pin_3)
- net Earth: now also J1.2 (Pin_2); no longer U10.9 (Adr0)
- net INPUT_3: now reaches R23.1
- net INPUT_3: now also J2.3 (Pin_3)
- net INPUT_4: now reaches R36.1
- net INPUT_4: now also J2.4 (Pin_4)
- net INPUT_1: now reaches R21.1
- net INPUT_1: now also J2.1 (Pin_1)
- net INPUT_2: now reaches R38.1
- net INPUT_2: now also J2.2 (Pin_2)
- net +3.3V renamed VCC
- net VCC: now also J1.4 (Pin_4)
- net I2C0_SCL renamed SCL
- net SCL: now also J1.5 (Pin_5)
- net I2C0_SDA renamed SDA
- net SDA: now also J1.6 (Pin_6)
- new net ADDR: J2.6 (Pin_6), U10.9 (Adr0)
- no-connect marks 0 -> 1
Other:
- moved on the sheet: C27, C31, U9E
