File: hardware/EuroPi-X/development/panelised.kicad_pcb (KiCad board)
At the start: 2 copper layers, 20.3 x 33 mm, 52 parts, among them J1 Conn_01x06_Pin, J2 Conn_01x06_Pin, J8 Conn_01x06_Pin, J9 Conn_01x06_Pin, U1 LM4040DBZ-10, U1 TL074, U2 MCP6004, U3 MCP3428

Commit message: save
Parts:
- added C1: 2.2uF, Capacitor_SMD:C_0805_2012Metric, F.Cu at (4.47, 63.2)
- added C2: 2.2uF, Capacitor_SMD:C_0805_2012Metric, F.Cu at (4.47, 46.6)
- added C3: 10uF, Capacitor_SMD:C_0805_2012Metric, F.Cu at (6.86, 65.2)
- added C4: 2.2uF, Capacitor_SMD:C_0805_2012Metric, F.Cu at (6.86, 44.6)
- added C5: 2.2uF, Capacitor_SMD:C_0805_2012Metric, F.Cu at (6.86, 48.6)
- added C6: 10uF, Capacitor_SMD:C_0805_2012Metric, F.Cu at (6.86, 61.2)
- added DS1: OLED-128O064D, allen-synthesis:KH-FPC0.5-H2.0SMT-30P-QCH FPC Connector 30 pin, F.Cu at (14.2, 54.8)
- added J1: Conn_01x08_Male, Connector_PinHeader_2.54mm:PinHeader_1x08_P2.54mm_Vertical_SMD_Pin1Left, F.Cu at (0.00, 54.6)
- added J2: Conn_01x02_Pin, Connector_PinHeader_2.54mm:PinHeader_1x02_P2.54mm_Vertical_SMD_Pin1Right, F.Cu at (16.5, 71.1)
- added J3: Conn_01x02_Pin, Connector_PinHeader_2.54mm:PinHeader_1x02_P2.54mm_Vertical_SMD_Pin1Right, F.Cu at (16.5, 38.0)
- added JP1: Close for I2C, Jumper:SolderJumper-2_P1.3mm_Bridged_RoundedPad1.0x1.5mm, F.Cu at (6.60, 40.8)
- added JP2: Close for I2C, Jumper:SolderJumper-2_P1.3mm_Bridged_RoundedPad1.0x1.5mm, F.Cu at (6.60, 37.0)
- added R1: 10K, Resistor_SMD:R_0603_1608Metric, F.Cu at (5.71, 51.6)
- added R2: 10K, Resistor_SMD:R_0603_1608Metric, F.Cu at (5.71, 53.8)
- added R3: 10K, Resistor_SMD:R_0603_1608Metric, F.Cu at (5.71, 56.0)
- added R4: 330K, Resistor_SMD:R_0603_1608Metric, F.Cu at (5.71, 58.1)
Routing:
- net +3V3: track 0.00 -> 60.6 mm, vias 0 -> 2
- net /D1/MOSI/SDA_3.3V: track 0.00 -> 41.4 mm, vias 0 -> 3
- net Net-(DS1-D2): track 0.00 -> 25.1 mm, vias 0 -> 2
- net /DC/SA0_3.3V: track 0.00 -> 16.2 mm, vias 0 -> 2
- net Net-(DS1-BS1): track 0.00 -> 15.8 mm
- net GND: track 0.00 -> 15.0 mm, vias 0 -> 8
- net /RST_3.3V: track 0.00 -> 14.8 mm, vias 0 -> 2
- net /D0/SCLK/SCK_3.3V: track 0.00 -> 13.1 mm
- net /CS_3.3V: track 0.00 -> 12.4 mm
- net Net-(DS1-C2N): track 0.00 -> 6.56 mm
- net Net-(DS1-VCC): track 0.00 -> 5.65 mm
- net Net-(DS1-C2P): track 0.00 -> 5.55 mm
- net Net-(DS1-IREF): track 0.00 -> 5.44 mm
- net Net-(DS1-VCOMH): track 0.00 -> 4.96 mm
- net Net-(DS1-C1P): track 0.00 -> 4.88 mm
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- added copper zone on B.Cu, net GND
- added copper zone on F.Cu, net GND
Other:
- board size 20.3 x 33 mm -> 23 x 75.8 mm
- board text added: "+3V3"
- board text added: "Address is 0x3D"
- board text added: "CS"
- board text added: "DC"
- board text added: "Enoki!"
- board text added: "For I2C, jump JP1 & JP2!"
- board text added: "RST"
- board text added: "SCK"
- board text added: "SSD1306 1.3{dblquote} Display Breakout board Toadstool Tech 2023"
