File: hardware/EuroPi-X/kicad/EuroPi-X.kicad_sch (KiCad schematic)
At the start: 164 parts, among them J1 Conn_01x16_Pin, J10 Thonkiconn_Mono_Jack, J11 Conn_02x08_Odd_Even, J12 Thonkiconn_Mono_Jack, J13 Thonkiconn_Mono_Jack, J14 Thonkiconn_Mono_Jack, J15 Thonkiconn_Mono_Jack, J16 Thonkiconn_Mono_Jack, J17 Thonkiconn_Mono_Jack, J18 Conn_01x03_Pin, J2 Conn_01x16_Pin, J22 Conn_01x11_Pin, J3 Thonkiconn_Mono_Jack, J4 Thonkiconn_Mono_Jack, J5 Conn_01x16_Pin, J6 Thonkiconn_Mono_Jack, J7 Thonkiconn_Mono_Jack, J8 Conn_01x16_Pin, J9 Thonkiconn_Mono_Jack, P1 USB_C_Plug_USB2.0, P2 Potentiometer_9mm_Vertical_Li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, P3 Potentiometer_9mm_Vertical_Li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, Q1 BSS138, SW1 B1, SW2 B2, U1 MCP6002-xSN, U10 MCP3428, U11 L7805, U12 LM4040DBZ-4.1, U2 LM4040DBZ-2.0, U3 LM4040DBZ-10, U4 RP2040, U7 TL074, U8 TL074, U9 MCP6004, Y1 Crystal_GND2

Commit message: add led on gp25
Parts:
- added D7: LED, symbol Device:LED
- added R62: 200R, Resistor_SMD:R_0402_1005Metric, symbol Device:R
Connections:
- net Earth: now also D7.1 (K)
- net GPIO_25_LED: now reaches U4.37 (GPIO25)
- net GPIO_25_LED: now also R62.1
- new net: D7.2 (A), R62.2
- no-connect marks 28 -> 27
Changed lines of the file:
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@@
   (no_connect (at 171.45 414.02))
   (no_connect (at 420.37 411.48))
-  (no_connect (at 168.91 278.13))
   (no_connect (at 659.13 203.2))
   (no_connect (at 511.81 461.01))
@@
     (stroke (width 0) (type default))
   )
+  (wire (pts (xy 148.59 314.96) (xy 152.4 314.96))
+    (stroke (width 0) (type default))
+  )
   (wire (pts (xy 443.23 149.86) (xy 440.69 149.86))
     (stroke (width 0) (type default))
@@
     (stroke (width 0) (type default))
   )
+  (wire (pts (xy 168.91 278.13) (xy 173.99 278.13))
+    (stroke (width 0) (type default))
+  )
   (wire (pts (xy 424.18 83.82) (xy 433.07 83.82))
     (stroke (width 0) (type default))
@@
     (stroke (width 0) (type default))
   )
+  (wire (pts (xy 175.26 318.77) (xy 175.26 314.96))
+    (stroke (width 0) (type default))
+  )
   (wire (pts (xy 476.25 438.15) (xy 468.63 438.15))
     (stroke (width 0) (type default))
@@
     (stroke (width 0) (type default))
   )
+  (wire (pts (xy 175.26 314.96) (xy 171.45 314.96))
+    (stroke (width 0) (type default))
+  )
   (wire (pts (xy 337.82 120.65) (xy 337.82 121.92))
     (stroke (width 0) (type default))
@@
     (stroke (width 0) (type default))
   )
+  (wire (pts (xy 160.02 314.96) (xy 163.83 314.96))
+    (stroke (width 0) (type default))
+  )
   (wire (pts (xy 377.19 416.56) (xy 381 416.56))
     (stroke (width 0) (type default))
@@
     (effects (font (size 1.27 1.27)) (justify left bottom))
   )
+  (label "GPIO_25_LED" (at 148.59 314.96 180) (fields_autoplaced)
+    (effects (font (size 1.27 1.27)) (justify right bottom))
+  )
   (label "SWCLK" (at 111.76 280.67 180) (fields_autoplaced)
     (effects (font (size 1.27 1.27)) (justify right bottom))
@@
     (effects (font (size 1.27 1.27)) (justify right bottom))
   )
+  (label "GPIO_25_LED" (at 173.99 278.13 0) (fields_autoplaced)
+    (effects (font (size 1.27 1.27)) (justify left bottom))
+  )
   (label "CV_OUTPUT_6_FRONT" (at 419.1 453.39 90) (fields_autoplaced)
     (effects (font (size 1.27 1.27)) (justify left bottom))
@@
     )
   )
+  (symbol (lib_id "power:Earth") (at 175.26 318.77 0) (unit 1)
+    (in_bom yes) (on_board yes) (dnp no) (fields_autoplaced)
+    (property "Reference" "#PWR096" (at 175.26 325.12 0)
+      (effects (font (size 1.27 1.27)) hide)
+    )
+    (property "Value" "Earth" (at 175.26 322.58 0)
+      (effects (font (size 1.27 1.27)) hide)
+    )
+    (property "Footprint" "" (at 175.26 318.77 0)
+      (effects (font (size 1.27 1.27)) hide)
+    )
+    (property "Datasheet" "~" (at 175.26 318.77 0)
+      (effects (font (size 1.27 1.27)) hide)
+    )
+    (pin "1")
+    (instances
+      (project "EuroPi-X"
+        (path "/a1be51f2-61d0-4240-8665-f31cc7b044f7"
+          (reference "#PWR096") (unit 1)
+        )
+      )
+    )
+  )
   (symbol (lib_id "Switch:SW_Push") (at 552.45 231.14 0) (unit 1)
     (in_bom yes) (on_board yes) (dnp no) (fields_autoplaced)
@@
     )
   )
+  (symbol (lib_id "Device:R") (at 156.21 314.96 90) (unit 1)
+    (in_bom yes) (on_board yes) (dnp no) (fields_autoplaced)
+    (property "Reference" "R62" (at 156.21 309.88 90)
+      (effects (font (size 1.27 1.27)))
+    )
+    (property "Value" "200R" (at 156.21 312.42 90)
+      (effects (font (size 1.27 1.27)))
+    )
+    (property "Footprint" "Resistor_SMD:R_0402_1005Metric" (at 156.21 316.738 90)
+      (effects (font (size 1.27 1.27)) hide)
+    )
+    (property "Datasheet" "~" (at 156.21 314.96 0)
+      (effects (font (size 1.27 1.27)) hide)
+    )
+    (property "JLCPCB PART#" "" (at 156.21 314.96 0)
+      (effects (font (size 1.27 1.27)) hide)
+    )
+    (property "JLC" "C25087" (at 156.21 314.96 0)
+      (effects (font (size 1.27 1.27)) hide)
+    )
+    (pin "1")
+    (pin "2")
+    (instances
+      (project "EuroPi-X"
+        (path "/a1be51f2-61d0-4240-8665-f31cc7b044f7"
+          (reference "R62") (unit 1)
+        )
+      )
+    )
+  )
   (symbol (lib_id "power:+5V") (at 560.07 118.11 0) (unit 1)
     (in_bom yes) (on_board yes) (dnp no) (fields_autoplaced)
@@
         )
       )
+    )
+  )
+  (symbol (lib_id "Device:LED") (at 167.64 314.96 180) (unit 1)
+    (in_bom yes) (on_board yes) (dnp no) (fields_autoplaced)
+    (property "Reference" "D7" (at 169.2275 308.61 0)
+      (effects (font (size 1.27 1.27)))
+    )
+    (property "Value" "LED" (at 169.2275 311.15 0)
+      (effects (font (size 1.27 1.27)))
+    )
+    (property "Footprint" "" (at 167.64 314.96 0)
+      (effects (font (size 1.27 1.27)) hide)
+    )
+    (property "Datasheet" "~" (at 167.64 314.96 0)
+      (effects (font (size 1.27 1.27)) hide)
+    )
+    (property "JLC" "C2286" (at 167.64 314.96 0)
+      (effects (font (size 1.27 1.27)) hide)
+    )
+    (pin "1")
+    (pin "2")
+    (instances
+      (project "EuroPi-X"
+        (path "/a1be51f2-61d0-4240-8665-f31cc7b044f7"
+          (reference "D7") (unit 1)
+        )
+      )

Commit message: create output dev board
Connections:
- net Earth: now also DAC1.4 (~{LDAC}), DAC2.4 (~{LDAC})
- net DAC_1_RDY: no longer names the net of DAC1.5 (RDY/~{BSY})
- net DAC_2_RDY: no longer names the net of DAC2.5 (RDY/~{BSY})
- no-connect marks 27 -> 29
Changed lines of the file:
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@@
   (no_connect (at 168.91 267.97))
   (no_connect (at 168.91 250.19))
+  (no_connect (at 163.83 355.6))
   (no_connect (at 168.91 262.89))
   (no_connect (at 168.91 255.27))
   (no_connect (at 171.45 414.02))
   (no_connect (at 420.37 411.48))
+  (no_connect (at 85.09 355.6))
   (no_connect (at 659.13 203.2))
   (no_connect (at 511.81 461.01))
@@
     (stroke (width 0) (type default))
   )
+  (wire (pts (xy 163.83 353.06) (xy 158.75 353.06))
+    (stroke (width 0) (type default))
+  )
   (wire (pts (xy 373.38 400.05) (xy 377.19 400.05))
     (stroke (width 0) (type default))
@@
     (stroke (width 0) (type default))
   )
-  (wire (pts (xy 158.75 355.6) (xy 163.83 355.6))
-    (stroke (width 0) (type default))
-  )
   (wire (pts (xy 220.98 176.53) (xy 220.98 168.91))
     (stroke (width 0) (type default))
@@
     (stroke (width 0) (type default))
   )
-  (wire (pts (xy 80.01 355.6) (xy 85.09 355.6))
-    (stroke (width 0) (type default))
-  )
   (wire (pts (xy 400.05 388.62) (xy 400.05 400.05))
     (stroke (width 0) (type default))
@@
     (stroke (width 0) (type default))
   )
+  (wire (pts (xy 158.75 353.06) (xy 158.75 355.6))
+    (stroke (width 0) (type default))
+  )
   (wire (pts (xy 491.49 241.3) (xy 488.95 241.3))
     (stroke (width 0) (type default))
@@
     (stroke (width 0) (type default))
   )
+  (wire (pts (xy 85.09 353.06) (xy 80.01 353.06))
+    (stroke (width 0) (type default))
+  )
   (wire (pts (xy 160.02 162.56) (xy 165.1 162.56))
     (stroke (width 0) (type default))
@@
     (stroke (width 0) (type default))
   )
+  (wire (pts (xy 80.01 353.06) (xy 80.01 355.6))
+    (stroke (width 0) (type default))
+  )
   (wire (pts (xy 563.88 273.05) (xy 566.42 273.05))
     (stroke (width 0) (type default))
@@
     (effects (font (size 1.27 1.27)) (justify left bottom))
   )
-  (label "DAC_1_RDY" (at 80.01 355.6 180) (fields_autoplaced)
-    (effects (font (size 1.27 1.27)) (justify right bottom))
-  )
   (label "CV_OUTPUT_8" (at 725.17 464.82 180) (fields_autoplaced)
     (effects (font (size 1.27 1.27)) (justify right bottom))
@@
     (effects (font (size 1.27 1.27)) (justify left bottom))
   )
-  (label "DAC_2_RDY" (at 158.75 355.6 180) (fields_autoplaced)
-    (effects (font (size 1.27 1.27)) (justify right bottom))
-  )
   (label "USB_DETECT" (at 139.7 95.25 0) (fields_autoplaced)
     (effects (font (size 1.27 1.27)) (justify left bottom))
@@
     )
   )
+  (symbol (lib_id "power:Earth") (at 158.75 355.6 0) (mirror y) (unit 1)
+    (in_bom yes) (on_board yes) (dnp no) (fields_autoplaced)
+    (property "Reference" "#PWR097" (at 158.75 361.95 0)
+      (effects (font (size 1.27 1.27)) hide)
+    )
+    (property "Value" "Earth" (at 158.75 359.41 0)
+      (effects (font (size 1.27 1.27)) hide)
+    )
+    (property "Footprint" "" (at 158.75 355.6 0)
+      (effects (font (size 1.27 1.27)) hide)
+    )
+    (property "Datasheet" "~" (at 158.75 355.6 0)
+      (effects (font (size 1.27 1.27)) hide)
+    )
+    (pin "1")
+    (instances
+      (project "EuroPi-X"
+        (path "/a1be51f2-61d0-4240-8665-f31cc7b044f7"
+          (reference "#PWR097") (unit 1)
+        )
+      )
+    )
+  )
   (symbol (lib_id "Connector_Generic:Conn_02x08_Odd_Even") (at 641.35 290.83 180) (unit 1)
     (in_bom yes) (on_board yes) (dnp no) (fields_autoplaced)
@@
         )
       )
+    )
+  )
+  (symbol (lib_id "power:Earth") (at 80.01 355.6 0) (mirror y) (unit 1)
+    (in_bom yes) (on_board yes) (dnp no) (fields_autoplaced)
+    (property "Reference" "#PWR098" (at 80.01 361.95 0)
+      (effects (font (size 1.27 1.27)) hide)
+    )
+    (property "Value" "Earth" (at 80.01 359.41 0)
+      (effects (font (size 1.27 1.27)) hide)
+    )
+    (property "Footprint" "" (at 80.01 355.6 0)
+      (effects (font (size 1.27 1.27)) hide)
+    )
+    (property "Datasheet" "~" (at 80.01 355.6 0)
+      (effects (font (size 1.27 1.27)) hide)
+    )
+    (pin "1")
+    (instances
+      (project "EuroPi-X"
+        (path "/a1be51f2-61d0-4240-8665-f31cc7b044f7"
+          (reference "#PWR098") (unit 1)
+        )
+      )
