File: hardware/EuroPi-X/development/output stage/output stage.kicad_pcb (KiCad board)
At the start: 2 copper layers, 20.3 x 15.2 mm, 27 parts, among them J1 Conn_01x06_Pin, J2 Conn_01x06_Pin, U1 TL074

Commit message: save
Connections:
- C2 pad 2: /OUTPUT_1 -> Net-(C2-Pad2)
- C3 pad 2: /OUTPUT_2 -> Net-(C3-Pad2)
- C4 pad 2: /OUTPUT_3 -> Net-(C4-Pad2)
- C5 pad 2: /OUTPUT_4 -> Net-(C5-Pad2)
- R12 pad 2: Net-(R12-Pad2) -> Net-(C4-Pad2)
- R16 pad 2: Net-(R16-Pad2) -> Net-(C5-Pad2)
- R4 pad 2: Net-(R4-Pad2) -> Net-(C2-Pad2)
- R8 pad 2: Net-(R8-Pad2) -> Net-(C3-Pad2)
- U1 pad 1: Net-(R4-Pad2) -> Net-(C2-Pad2)
- U1 pad 14: Net-(R16-Pad2) -> Net-(C5-Pad2)
- U1 pad 7: Net-(R8-Pad2) -> Net-(C3-Pad2)
- U1 pad 8: Net-(R12-Pad2) -> Net-(C4-Pad2)
Routing:
- net Net-(C3-Pad2): track 0.00 -> 3.78 mm
- net Net-(C2-Pad2): track 0.00 -> 3.78 mm
- net Net-(C5-Pad2): track 0.00 -> 3.78 mm
- net Net-(C4-Pad2): track 0.00 -> 3.78 mm
- net Net-(R8-Pad2): track 2.10 -> 0.00 mm
- net Net-(R4-Pad2): track 2.10 -> 0.00 mm
- net Net-(R16-Pad2): track 2.09 -> 0.00 mm
- net Net-(R12-Pad2): track 2.09 -> 0.00 mm
- net /OUTPUT_3: track 24.6 -> 23.1 mm
- net /OUTPUT_4: track 20.8 -> 19.9 mm
- net /OUTPUT_2: track 7.36 -> 8.16 mm
- net /OUTPUT_1: track 7.36 -> 7.97 mm

Commit message: save
Parts:
- moved DAC1 0.25 mm to (12.1, 12.7)
- moved J1 0.25 mm to (1.27, 1.27)
- moved C1 0.25 mm to (15.2, 10.2)
- moved C2 0.25 mm to (15.2, 7.62)
- moved C3 0.25 mm to (15.2, 2.54)
- moved C4 0.25 mm to (5.08, 2.54)
- moved C5 0.25 mm to (5.08, 7.62)
- moved C6 0.25 mm to (15.2, 5.08)
- moved C7 0.25 mm to (5.08, 5.08)
- moved R1 0.25 mm to (5.08, 10.4)
- moved R10 0.25 mm to (7.62, 13.0)
- moved R11 0.25 mm to (5.08, 3.81)
- moved R12 0.25 mm to (5.08, 1.27)
- moved R13 0.25 mm to (5.08, 14.2)
- moved R14 0.25 mm to (7.62, 14.2)
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Other:
- outline, holes or cut-outs redrawn
